Commit message: Added sim_controller and simulation code for testing during simulation

File: src/dual_proxy_motion_robot/panda_arm.urdf (robot description, URDF)
Before this commit: robot panda, 9 links, 8 joints
Links:
- added link camera_link, mass 0.1; collision sphere radius=0.01; visual mesh filename=../../../model/panda/meshes/realsense_d455/realsense1.obj
- added link eef_2, mass 0.001; collision sphere radius=0.01; visual sphere radius=0.01
Joints:
- added joint joint_camera: type fixed, parent eef_2, child camera_link, origin xyz=0.0 0.0 0.21  rpy=-1.57 0.0 -0.7853
- added joint joint_fixed_eef2: type fixed, parent link7, child eef_2, origin xyz=0.0 0.0 0.12 rpy=0 0 -0.78539816339
